Commit message: feat: complete phase 8 nav2 visual navigation

File: ros2_ws/src/nova_carter_bringup/urdf/nova_carter.urdf.xacro (robot description, xacro)
@@ -2,5 +2,19 @@
 <robot xmlns:xacro="http://www.ros.org/wiki/xacro" name="nova_carter">
   <!-- Values were extracted from the composed Isaac Sim 6.0 Nova Carter USD. -->
-  <link name="base_link"/>
+  <material name="nova_dark"><color rgba="0.12 0.15 0.18 1"/></material>
+  <material name="nova_green"><color rgba="0.20 0.75 0.35 1"/></material>
+  <material name="wheel_black"><color rgba="0.025 0.025 0.025 1"/></material>
+  <link name="base_link">
+    <visual>
+      <origin xyz="-0.2335 0 0.34" rpy="0 0 0"/>
+      <geometry><box size="0.747 0.50 0.40"/></geometry>
+      <material name="nova_dark"/>
+    </visual>
+    <visual>
+      <origin xyz="0.02 0 0.58" rpy="0 0 0"/>
+      <geometry><box size="0.20 0.32 0.10"/></geometry>
+      <material name="nova_green"/>
+    </visual>
+  </link>
   <link name="front_stereo_camera_link"/>
   <link name="front_stereo_camera_left_optical"/>
@@ -23,5 +37,10 @@
     <origin xyz="0 -0.0197 0.0061" rpy="0 1.57079632679 0"/>
   </joint>
-  <link name="wheel_left"/><link name="wheel_right"/>
+  <link name="wheel_left">
+    <visual><geometry><cylinder radius="0.14" length="0.06"/></geometry><material name="wheel_black"/></visual>
+  </link>
+  <link name="wheel_right">
+    <visual><geometry><cylinder radius="0.14" length="0.06"/></geometry><material name="wheel_black"/></visual>
+  </link>
   <joint name="joint_wheel_left" type="continuous">
     <parent link="base_link"/><child link="wheel_left"/>

Commit message: feat: complete phase 9 dynamic visual navigation

File: ros2_ws/src/nova_carter_bringup/urdf/nova_carter.urdf.xacro (robot description, xacro)
@@ -36,4 +36,51 @@
     <parent link="front_stereo_camera_link"/><child link="front_stereo_camera_imu"/>
     <origin xyz="0 -0.0197 0.0061" rpy="0 1.57079632679 0"/>
+  </joint>
+  <!-- Stage 9 surround Hawk baselines.  The midpoint poses and rotations are
+       extracted from the local Isaac Sim 6.0.1 nova_carter.usd. -->
+  <link name="left_stereo_camera_link"/>
+  <link name="left_stereo_camera_left_optical"/>
+  <link name="left_stereo_camera_right_optical"/>
+  <joint name="left_stereo_mount" type="fixed">
+    <parent link="base_link"/><child link="left_stereo_camera_link"/>
+    <origin xyz="-0.35543 0.15 0.3459" rpy="0 0 1.57079632679"/>
+  </joint>
+  <joint name="left_stereo_left_optical_joint" type="fixed">
+    <parent link="left_stereo_camera_link"/><child link="left_stereo_camera_left_optical"/>
+    <origin xyz="0 0.075 0" rpy="-1.57079632679 0 -1.57079632679"/>
+  </joint>
+  <joint name="left_stereo_right_optical_joint" type="fixed">
+    <parent link="left_stereo_camera_link"/><child link="left_stereo_camera_right_optical"/>
+    <origin xyz="0 -0.075 0" rpy="-1.57079632679 0 -1.57079632679"/>
+  </joint>
+  <link name="right_stereo_camera_link"/>
+  <link name="right_stereo_camera_left_optical"/>
+  <link name="right_stereo_camera_right_optical"/>
+  <joint name="right_stereo_mount" type="fixed">
+    <parent link="base_link"/><child link="right_stereo_camera_link"/>
+    <origin xyz="-0.35544 -0.15 0.3459" rpy="0 0 -1.57079632679"/>
+  </joint>
+  <joint name="right_stereo_left_optical_joint" type="fixed">
+    <parent link="right_stereo_camera_link"/><child link="right_stereo_camera_left_optical"/>
+    <origin xyz="0 0.075 0" rpy="-1.57079632679 0 -1.57079632679"/>
+  </joint>
+  <joint name="right_stereo_right_optical_joint" type="fixed">
+    <parent link="right_stereo_camera_link"/><child link="right_stereo_camera_right_optical"/>
+    <origin xyz="0 -0.075 0" rpy="-1.57079632679 0 -1.57079632679"/>
+  </joint>
+  <link name="back_stereo_camera_link"/>
+  <link name="back_stereo_camera_left_optical"/>
+  <link name="back_stereo_camera_right_optical"/>
+  <joint name="back_stereo_mount" type="fixed">
+    <parent link="base_link"/><child link="back_stereo_camera_link"/>
+    <origin xyz="-0.5637 0.000002 0.3459" rpy="0 0 3.14159265359"/>
+  </joint>
+  <joint name="back_stereo_left_optical_joint" type="fixed">
+    <parent link="back_stereo_camera_link"/><child link="back_stereo_camera_left_optical"/>
+    <origin xyz="0 0.075 0" rpy="-1.57079632679 0 -1.57079632679"/>
+  </joint>
+  <joint name="back_stereo_right_optical_joint" type="fixed">
+    <parent link="back_stereo_camera_link"/><child link="back_stereo_camera_right_optical"/>
+    <origin xyz="0 -0.075 0" rpy="-1.57079632679 0 -1.57079632679"/>
   </joint>
   <link name="wheel_left">
